File: PowerPCB/PowerPCB.kicad_pcb (KiCad board)
At the start: 2 copper layers, 78 x 70 mm, 25 parts, among them J2 Conn_01x02_Pin, J3 Conn_01x02_Pin, J4 Conn_01x02_Pin, J5 Conn_01x04_Pin, J6 Conn_01x02_Pin, J7 Conn_01x02_Pin, Q1 BS170, Q2 BS170

Commit message: ?
Parts:
- removed REF**: MountingHole_4.3mm_M4, MountingHole:MountingHole_4.3mm_M4
- removed REF** (x3): MountingHole_4mm, MountingHole:MountingHole_4mm
- added D5: 1N4007, Diode_THT:D_DO-41_SOD81_P10.16mm_Horizontal, F.Cu at (119.7, 84.8)
- added D6: 1N4007, Diode_THT:D_DO-41_SOD81_P10.16mm_Horizontal, F.Cu at (107.9, 50.3)
- added F1: Fuse, Meloen:RB500-50, F.Cu at (111.3, 79.0)
- added F2: Fuse, Meloen:RB500-50, F.Cu at (113.4, 40.7)
- added G***: LOGO, Logo:Logo_100x78, B.Cu at (94.3, 60.1)
- added H1: MountingHole, MountingHole:MountingHole_3.2mm_M3, F.Cu at (124.6, 34.3)
- added H2: MountingHole, MountingHole:MountingHole_3.2mm_M3, F.Cu at (124.6, 91.3)
- added H3: MountingHole, MountingHole:MountingHole_3.2mm_M3, F.Cu at (59.6, 91.3)
- added H4: MountingHole, MountingHole:MountingHole_3.2mm_M3, F.Cu at (59.6, 34.3)
- J7, Supercaps1: moved to F.Cu
- moved J7 5.46 mm to (110.8, 94.7), turned to 0 degrees
- moved Supercaps1 4.89 mm to (127.0, 49.8), turned to 90 degrees
Connections:
- Buckboost1 pad 2: buckboostgrnd -> GND
- Supercaps1 pad 1: Supercap+ -> Net-(Supercaps1-Pin_1)
- Supercaps1 pad 2: Supercap- -> GND
- U1 pad 1: 24V -> Net-(D5-K)
- U1 pad 2: buckboostgrnd -> GND
- U2 pad 2: Supercap- -> unconnected-(U2-IN--Pad2)
- U3 pad 2: Supercap- -> GND
Routing:
- net Supercap-: track 32.7 -> 0.00 mm
- net Net-(D5-K): track 0.00 -> 21.3 mm
- net Supercap+: track 32.8 -> 46.9 mm
- net Net-(Supercaps1-Pin_1): track 0.00 -> 12.1 mm
- net buckboostgrnd: track 9.77 -> 0.00 mm
- net 24V: track 44.4 -> 53.2 mm
- net Net-(J7-Pin_1): track 61.4 -> 59.3 mm
