File: PowerPCB/PowerPCB.kicad_sch (KiCad schematic)
At the start: 7 parts, among them J1 Conn_01x02_Pin, J2 Conn_01x02_Pin, J3 Conn_01x02_Pin, J4 Conn_01x02_Pin

Commit message: PowerPCB
Parts:
- added C1, C2, C3: C, Capacitor_THT:CP_Radial_D5.0mm_P2.50mm, symbol Device:C
- added D2: 1N4007, Diode_THT:D_DO-41_SOD81_P10.16mm_Horizontal, symbol Diode:1N4007
- added J5: Conn_01x04_Pin, Meloen:Audio jack, symbol Connector:Conn_01x04_Pin
- added J6, J7: Conn_01x02_Pin, Connector_Phoenix_MSTB:PhoenixContact_MSTBA_2,5_2-G-5,08_1x02_P5.08mm_Horizontal, symbol Connector:Conn_01x02_Pin
- added Q1, Q2: BS170, Package_TO_SOT_THT:TO-92_Inline, symbol Transistor_FET:BS170
- added R1, R2: 100, Resistor_THT:R_Axial_DIN0204_L3.6mm_D1.6mm_P7.62mm_Horizontal, symbol Device:R
- added R3, R4: 10k, Resistor_THT:R_Axial_DIN0204_L3.6mm_D1.6mm_P7.62mm_Horizontal, symbol Device:R
- added Supercaps1: Supercaps, Connector_Phoenix_MSTB:PhoenixContact_MSTBA_2,5_2-G-5,08_1x02_P5.08mm_Horizontal, symbol Connector:Conn_01x02_Pin
- Buckboost1: renamed from J1; value Conn_01x02_Pin -> Buckboost; footprint (none) -> Connector_Phoenix_MSTB:PhoenixContact_MSTBA_2,5_2-G-5,08_1x02_P5.08mm_Horizontal
- J2, J3, J4: footprint (none) -> Connector_Phoenix_MSTB:PhoenixContact_MSTBA_2,5_2-G-5,08_1x02_P5.08mm_Horizontal
- U1, U2, U3: footprint (none) -> Meloen:LM2596_module_opvoetjes
Connections:
- net 24V: now also D2.1 (K), J6.2 (Pin_2), J7.2 (Pin_2); no longer U2.1 (IN+), U3.1 (IN+)
- net GND: now also C1.2, C2.2, C3.2, J5.4 (Pin_4), Q1.3 (S), Q2.3 (S), R3.2, R4.2
- net buckboostgrnd: no longer U2.2 (IN-), U3.2 (IN-)
- net at J3.2 (Pin_2), U2.4 (OUT+): now also C2.1
- net at J4.2 (Pin_2), U3.4 (OUT+): now also C1.1
- net at J2.2 (Pin_2), U1.4 (OUT+): now also C3.1
- new net: Q2.2 (G), R2.2
- new net: Q1.2 (G), R1.2
- new net: D2.2 (A), J6.1 (Pin_1), Q1.1 (D), R3.1
- new net: J7.1 (Pin_1), Q2.1 (D), R4.1
- new net Supercap+: Supercaps1.1 (Pin_1), U2.1 (IN+), U3.1 (IN+)
- new net Supercap-: Supercaps1.2 (Pin_2), U2.2 (IN-), U3.2 (IN-)
- new net Transistor magneet: J5.2 (Pin_2), R1.1
- new net Transistor metaal: J5.1 (Pin_1), R2.1
- no-connect marks 0 -> 1
Other:
- moved on the sheet: Buckboost1

Commit message: ?
Parts:
- added D5, D6: 1N4007, Diode_THT:D_DO-41_SOD81_P10.16mm_Horizontal, symbol Diode:1N4007
- added F1, F2: Fuse, Meloen:RB500-50, symbol Device:Fuse
- added H1, H2, H3, H4: MountingHole, MountingHole:MountingHole_3.2mm_M3, symbol Mechanical:MountingHole
Connections:
- net buckboostgrnd is gone; now on net GND: Buckboost1.2 (Pin_2), U1.2 (IN-)
- net 24V: now also F1.1; no longer U1.1 (IN+)
- net GND: now also Supercaps1.2 (Pin_2), U3.2 (IN-), D5.2 (A), D6.2 (A)
- net Supercap+: now also D6.1 (K), F2.2; no longer Supercaps1.1 (Pin_1)
- removed net Supercap-: Supercaps1.2 (Pin_2), U2.2 (IN-), U3.2 (IN-)
- new net: F2.1, Supercaps1.1 (Pin_1)
- new net: D5.1 (K), F1.2, U1.1 (IN+)
