File: RoverPCB/RoverPCB.kicad_sch (KiCad schematic)
At the start: 3 parts, among them J1 Conn_01x02

Commit message: PCBs
Parts:
- removed U2: ~, Zuydlib3:LM2596_module, symbol Zuydlib3:LM2596_module
- added J10, J2, J3, J6, J7, J9: Conn_01x04_Pin, Meloen:Audio jack, symbol Connector:Conn_01x04_Pin
- added J12: I2C 3V3, Meloen:Audio jack, symbol Connector:Conn_01x04_Pin
- added J13, J15, J16, J17: I2C, Meloen:Audio jack, symbol Connector:Conn_01x04_Pin
- added J14: UART, Meloen:Audio jack, symbol Connector:Conn_01x04_Pin
- added J4: PWM bord, Connector_PinHeader_2.54mm:PinHeader_1x06_P2.54mm_Vertical, symbol Connector:Conn_01x06_Pin
- added J5: Conn_01x15_Socket, Connector_PinHeader_2.54mm:PinHeader_1x15_P2.54mm_Vertical, symbol Connector:Conn_01x15_Socket
- added J8: Conn_01x04_Pin, symbol Connector:Conn_01x04_Pin
- added R1, R2, R3, R4: R, Resistor_THT:R_Axial_DIN0204_L3.6mm_D1.6mm_P7.62mm_Horizontal, symbol Device:R
Connections:
- net +3V3: now also J12.1 (Pin_1), J2.2 (Pin_2), J2.3 (Pin_3), J3.2 (Pin_2), J3.3 (Pin_3)
- net +5V: now also J1.2 (Pin_2), J13.1 (Pin_1), J14.1 (Pin_1), J15.1 (Pin_1), J16.1 (Pin_1), J17.1 (Pin_1), J4.1 (Pin_1), J4.2 (Pin_2)
- net GND: now also J1.1 (Pin_1), J10.4 (Pin_4), J12.4 (Pin_4), J13.4 (Pin_4), J14.4 (Pin_4), J15.4 (Pin_4), J16.4 (Pin_4), J17.4 (Pin_4), J4.6 (Pin_6), J6.4 (Pin_4), J7.4 (Pin_4), J8.4 (Pin_4), J9.4 (Pin_4), R1.2, R2.2, R3.2, R4.2
- net SDA: now reaches U1.11 (D21)
- net SDA: now also J12.3 (Pin_3), J13.3 (Pin_3), J15.3 (Pin_3), J16.3 (Pin_3), J17.3 (Pin_3), J4.3 (Pin_3)
- net RX: now reaches U1.12 (RX0)
- net RX: now also J14.3 (Pin_3)
- net TX: now reaches U1.13 (TX0)
- net TX: now also J14.2 (Pin_2)
- net SCL: now reaches U1.14 (D22)
- net SCL: now also J12.2 (Pin_2), J13.2 (Pin_2), J15.2 (Pin_2), J16.2 (Pin_2), J17.2 (Pin_2), J4.4 (Pin_4)
- net Button2: now reaches U1.20 (D35)
- net Button2: now also J3.1 (Pin_1), R4.1
- net LDR2: now reaches U1.21 (D32)
- net LDR2: now also J3.4 (Pin_4), R3.1
- net Button1: now reaches U1.22 (D33)
- net Button1: now also J2.1 (Pin_1), R2.1
- net LDR1: now reaches U1.23 (D25)
- net LDR1: now also J2.4 (Pin_4), R1.1
- new net: J10.1 (Pin_1), J5.1 (Pin_1)
- new net: J10.2 (Pin_2), J5.2 (Pin_2)
- new net: J10.3 (Pin_3), J5.3 (Pin_3)
- new net: J5.13 (Pin_13), J6.1 (Pin_1)
- new net: J5.14 (Pin_14), J6.2 (Pin_2)
- new net: J5.15 (Pin_15), J6.3 (Pin_3)
- new net: J5.10 (Pin_10), J7.1 (Pin_1)
- new net: J5.11 (Pin_11), J7.2 (Pin_2)
- new net: J5.12 (Pin_12), J7.3 (Pin_3)
- new net: J5.4 (Pin_4), J9.1 (Pin_1)
- new net: J5.5 (Pin_5), J9.2 (Pin_2)
- new net: J5.6 (Pin_6), J9.3 (Pin_3)
- new net: J5.7 (Pin_7), J8.1 (Pin_1)
- new net: J5.8 (Pin_8), J8.2 (Pin_2)
- new net: J5.9 (Pin_9), J8.3 (Pin_3)
- no-connect marks 0 -> 1
Other:
- moved on the sheet: J1

Commit message: PCBRover final
Parts:
- removed J17: I2C, Meloen:Audio jack, symbol Connector:Conn_01x04_Pin
- added H1: MountingHole_Pad, MountingHole:MountingHole_4mm_Pad, symbol Mechanical:MountingHole_Pad
- added J11: arm, Meloen:Audio jack, symbol Connector:Conn_01x04_Pin
- added R5: R, Resistor_THT:R_Axial_DIN0204_L3.6mm_D1.6mm_P7.62mm_Horizontal, symbol Device:R
- added SW1: SW_DPDT_x2, Zuydlib4:SW_CuK_SPDT_Angled, symbol Switch:SW_DPDT_x2
- J1: value Conn_01x02 -> Voeding
- J10: value Conn_01x04_Pin -> ExtraPWM2
- J2: value Conn_01x04_Pin -> Left solartacker
- J3: value Conn_01x04_Pin -> Right solartracker
- J6: value Conn_01x04_Pin -> Motor1
- J7: value Conn_01x04_Pin -> Motor2
- J8: value Conn_01x04_Pin -> Motor3; footprint (none) -> Meloen:Audio jack
- J9: value Conn_01x04_Pin -> extraPWM1
- U1: footprint Meloen:ESP32_DEVKIT_V1_op_voetjes -> Meloen:ESP32_DEVKIT_V1_op_voetjes2rij
Connections:
- net +5V: now also SW1.1 (A); no longer J1.2 (Pin_2)
- net GND: now also H1.1, J11.4 (Pin_4), R5.1
- net RX: now also U1.6 (RX2); no longer U1.12 (RX0)
- net TX: now also U1.7 (TX2); no longer U1.13 (TX0)
- net Transistor metaal: now reaches U1.10 (D19)
- net Transistor metaal: now also J11.1 (Pin_1)
- net Metaal detector: now reaches U1.8 (D5)
- net Metaal detector: now also J11.3 (Pin_3), R5.2
- net Transistor magneet: now reaches U1.9 (D18)
- net Transistor magneet: now also J11.2 (Pin_2)
- new net: J1.2 (Pin_2), SW1.2 (B)
- no-connect marks 1 -> 2

Commit message: PowerPCB
Parts:
- removed H1: MountingHole_Pad, MountingHole:MountingHole_4mm_Pad, symbol Mechanical:MountingHole_Pad
Changed lines of the file:
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@@
-	(symbol
-		(lib_id "power:GND")
-		(at 157.48 46.99 0)
-		(unit 1)
-		(exclude_from_sim no)
-		(in_bom yes)
-		(on_board yes)
-		(dnp no)
-		(fields_autoplaced yes)
-		(property "Reference" "#PWR026"
-			(at 157.48 53.34 0)
-			(effects
-				(font
-					(size 1.27 1.27)
-				)
-				(hide yes)
-			)
-		)
-		(property "Value" "GND"
-			(at 157.48 52.07 0)
-			(effects
-				(font
-					(size 1.27 1.27)
-				)
-			)
-		)
-		(property "Footprint" ""
-			(at 157.48 46.99 0)
-			(effects
-				(font
-					(size 1.27 1.27)
-				)
-				(hide yes)
-			)
-		)
-		(property "Datasheet" ""
-			(at 157.48 46.99 0)
-			(effects
-				(font
-					(size 1.27 1.27)
-				)
-				(hide yes)
-			)
-		)
-		(property "Description" "Power symbol creates a global label with name \"GND\" , ground"
-			(at 157.48 46.99 0)
-			(effects
-				(font
-					(size 1.27 1.27)
-				)
-				(hide yes)
-			)
-		)
-		(pin "1"
-		)
-		(instances
-			(project ""
-				(path "/cccc5dfb-8b1f-48a4-a5eb-15bc94ab9727"
-					(reference "#PWR026")
-					(unit 1)
-				)
-			)
-		)
-	)
 	(symbol
 		(lib_id "power:GND")
@@
 					(unit 1)
 				)
-			)
-		)
-	)
-	(symbol
-		(lib_id "Mechanical:MountingHole_Pad")
-		(at 157.48 44.45 0)
-		(unit 1)
-		(exclude_from_sim no)
-		(in_bom no)
-		(on_board yes)
-		(dnp no)
-		(fields_autoplaced yes)
-		(property "Reference" "H1"
-			(at 160.02 41.9099 0)
-			(effects
-				(font
-					(size 1.27 1.27)
-				)
-				(justify left)
-			)
-		)
-		(property "Value" "MountingHole_Pad"
-			(at 160.02 44.4499 0)
-			(effects
-				(font
-					(size 1.27 1.27)
-				)
-				(justify left)
-			)
-		)
-		(property "Footprint" "MountingHole:MountingHole_4mm_Pad"
-			(at 157.48 44.45 0)
-			(effects
-				(font
-					(size 1.27 1.27)
-				)
-				(hide yes)
-			)
-		)
-		(property "Datasheet" "~"
-			(at 157.48 44.45 0)
-			(effects
-				(font
-					(size 1.27 1.27)
-				)
-				(hide yes)
-			)
-		)
-		(property "Description" "Mounting Hole with connection"
-			(at 157.48 44.45 0)
-			(effects
-				(font
-					(size 1.27 1.27)
-				)
-				(hide yes)
-			)
-		)
-		(pin "1"
-		)
-		(instances
-			(project ""
-				(path "/cccc5dfb-8b1f-48a4-a5eb-15bc94ab9727"
-					(reference "H1")
-					(unit 1)
-				)

Commit message: ?
Parts:
- added H1, H2, H3, H4: MountingHole, MountingHole:MountingHole_3.2mm_M3, symbol Mechanical:MountingHole
- added J17, J18: Conn_01x02, Connector_PinHeader_2.54mm:PinHeader_1x02_P2.54mm_Vertical, symbol Connector_Generic:Conn_01x02
Connections:
- net +5V: now also J17.1 (Pin_1), J18.1 (Pin_1)
- net GND: now also J17.2 (Pin_2), J18.2 (Pin_2)
